Commit message: initial commit

File: robots/descriptions/go2_description/xacro/const.xacro (robot description, xacro)
@@ -19,8 +19,21 @@
     <xacro:property name="stick_radius" value="0.01"/>
     <xacro:property name="stick_length" value="0.2"/>
-    <!-- kinematic value -->
-    <xacro:property name="thigh_offset" value="0.0955"/>
+    <!-- processed_params.yaml: file to be created by the python file, to imitate domain randomazation -->
+    <xacro:arg name="config_yaml"
+            default="$(find sensor_data_collector_pkg)/config/robot_params/go2/processed_params.yaml"/>
+    <!-- YAML を読み込む（※ 非推奨警告に従い xacro.load_yaml を使用） -->
+    <xacro:property name="cfg" value="${xacro.load_yaml('$(arg config_yaml)')}"/>
+    <!-- YAML値をデフォルトとする「引数」 -->
+    <xacro:arg name="thigh_offset_arg" default="${cfg['kinematics']['thigh_offset']}"/>
+    <xacro:arg name="thigh_length_arg"  default="${cfg['kinematics']['thigh_length']}"/>
+    <xacro:arg name="calf_length_arg" default="${cfg['kinematics']['calf_length']}"/>
+    <!-- This reflects robot_length -->
+    <xacro:property name="thigh_offset" value="$(arg thigh_offset_arg)"/>
+    <xacro:property name="thigh_length" value="$(arg thigh_length_arg)"/>
+    <xacro:property name="calf_length" value="$(arg calf_length_arg)"/>
+    <!-- kinematic value is set by a yaml file -->
+    <!-- <xacro:property name="thigh_offset" value="0.0955"/>
     <xacro:property name="thigh_length" value="0.213"/>
-    <xacro:property name="calf_length" value="0.213"/>
+    <xacro:property name="calf_length" value="0.213"/> -->
     <!-- leg offset from trunk center value -->
     <xacro:property name="leg_offset_x" value="0.1934"/>

File: robots/descriptions/go2_description/xacro/gazebo.xacro (robot description, xacro)
@@ -11,5 +11,21 @@
         <xyz_offset>0 0 0</xyz_offset>
         <rpy_offset>0 0 0</rpy_offset>
-        <gaussian_noise>0.01</gaussian_noise>
+        <gaussian_noise>0.00</gaussian_noise>
+    </plugin>
+    </gazebo>
+    <!-- p3d plugin publishing ground-truth odom for imu_link -->
+    <gazebo>
+    <plugin filename="libgazebo_ros_p3d.so" name="p3d_imu_controller">
+        <ros>
+        <!-- Use a distinct namespace/topic so it doesn't collide with the base_link p3d -->
+        <namespace>/imu</namespace>
+        <argument>odom:=odom/ground_truth_imu</argument>
+        </ros>
+        <body_name>imu_link</body_name>
+        <frame_name>world</frame_name>
+        <update_rate>10.0</update_rate>
+        <xyz_offset>0 0 0</xyz_offset>
+        <rpy_offset>0 0 0</rpy_offset>
+        <gaussian_noise>0.0</gaussian_noise>
     </plugin>
     </gazebo>
@@ -22,5 +38,5 @@
         <sensor name="imu_sensor" type="imu">
             <always_on>true</always_on>
-            <update_rate>100</update_rate>
+            <update_rate>200</update_rate>
             <imu>
             <angular_velocity>
@@ -28,5 +44,5 @@
                 <noise type="gaussian">
                     <mean>0.0</mean>
-                    <stddev>2e-4</stddev>
+                    <stddev>1e-6</stddev>
                 </noise>
                 </x>
@@ -34,5 +50,5 @@
                 <noise type="gaussian">
                     <mean>0.0</mean>
-                    <stddev>2e-4</stddev>
+                    <stddev>1e-6</stddev>
                 </noise>
                 </y>
@@ -40,5 +56,5 @@
                 <noise type="gaussian">
                     <mean>0.0</mean>
-                    <stddev>2e-4</stddev>
+                    <stddev>1e-6</stddev>
                 </noise>
                 </z>
@@ -48,5 +64,5 @@
                 <noise type="gaussian">
                     <mean>0.0</mean>
-                    <stddev>1.7e-2</stddev>
+                    <stddev>1e-6</stddev>
                 </noise>
                 </x>
@@ -54,5 +70,5 @@
                 <noise type="gaussian">
                     <mean>0.0</mean>
-                    <stddev>1.7e-2</stddev>
+                    <stddev>1e-6</stddev>
                 </noise>
                 </y>
@@ -60,5 +76,5 @@
                 <noise type="gaussian">
                     <mean>0.0</mean>
-                    <stddev>1.7e-2</stddev>
+                    <stddev>1e-6</stddev>
                 </noise>
                 </z>

File: robots/descriptions/go2_description/xacro/leg.xacro (robot description, xacro)
@@ -128,5 +128,5 @@
             </inertial>
         </link>
-        <joint name="${name}_foot_joint" type="fixed">0
+        <joint name="${name}_foot_joint" type="fixed">
             <origin rpy="0 0 0" xyz="0 0 ${-(calf_length)}"/>
             <parent link="${name}_lower_leg_link"/>
@@ -155,4 +155,14 @@
             </inertial>
         </link>
+        <gazebo reference="${name}_foot_link">
+            <sensor type="contact" name="${name}_foot_contact">
+            <contact>
+                <collision>${name}_lower_leg_link_fixed_joint_lump__${name}_foot_link_collision_1</collision>
+                <topic>/${name}_foot_contact</topic>
+            </contact>
+            <always_on>1</always_on>
+            <update_rate>200</update_rate>
+            </sensor>
+        </gazebo>
         <ros2_control name="${name}" type="system">
             <hardware>
